File: Proj1/Proj1.kicad_sch (KiCad schematic)
At the start: 11 parts, among them SW1 SW_Push, SW2 SW_Push, SW3 SW_Push, SW4 SW_Push, SW5 SW_Push, SW7 RotaryEncoder_Switch_MP, U1 XIAO-RP2040-DIP

Commit message: The board is done!
Parts:
- removed D1, D2, D3: SK6812, LED_SMD:LED_SK6812_PLCC4_5.0x5.0mm_P3.2mm, symbol LED:SK6812
- added RC1: RotaryEncoder_Switch_MP, Rotary_Encoder:RotaryEncoder_Alps_EC11E-Switch_Vertical_H20mm_CircularMountingHoles, symbol Device:RotaryEncoder_Switch_MP
- OL1: footprint KBD:OLED -> Connector_PinHeader_2.54mm:PinHeader_1x04_P2.54mm_Vertical
- renumbered SW7 to RC2
Connections:
- net GND: now also RC1.C; no longer RC2.S2
- net at U1.1 (GPIO26/ADC0/A0): now also RC1.B; no longer RC2.A
- net at U1.2 (GPIO27/ADC1/A1): now also RC1.A; no longer RC2.B
- net at U1.3 (GPIO28/ADC2/A2): now also RC2.B; no longer RC2.S1
- net at U1.4 (GPIO29/ADC3/A3): now also RC2.A; no longer OL1.1 (SDA)
- net at U1.5 (GPIO6/SDA): now also OL1.1 (SDA); no longer OL1.2 (SCL)
- net at U1.6 (GPIO7/SCL): now also OL1.2 (SCL); no longer SW5.1
- net at U1.7 (GPIO0/TX): now also SW5.1
Other:
- moved on the sheet: OL1, RC2, SW1, SW2, SW3, SW4, SW5, U1
