File: Proj1/Proj1.kicad_pcb (KiCad board)
At the start: 2 copper layers, 73.5 x 72.5 mm, 14 parts, among them SW1 SW_Push, SW2 SW_Push, SW3 SW_Push, SW4 SW_Push, SW5 SW_Push, SW7 RotaryEncoder_Switch_MP, U1 XIAO-RP2040-DIP

Commit message: The board is done!
Parts:
- removed D1, D2, D3: SK6812, LED_SMD:LED_SK6812_PLCC4_5.0x5.0mm_P3.2mm
- added G***: LOGO, Logo:LogoT2H-5percent, F.Cu at (122.0, 91.5)
- added REF**: MountingHole_3.2mm_M3, MountingHole:MountingHole_3.2mm_M3, F.Cu at (75.0, 27.5)
- added SW6: RotaryEncoder_Switch_MP, Rotary_Encoder:RotaryEncoder_Alps_EC11E-Switch_Vertical_H20mm_CircularMountingHoles, F.Cu at (76.5, 36.5)
- OL1: footprint KBD:OLED -> Connector_PinHeader_2.54mm:PinHeader_1x04_P2.54mm_Vertical
- moved OL1 42.6 mm to (123.4, 27.0), turned to 90 degrees
- moved SW1 1.96 mm to (100.2, 54.9)
- moved SW2 1.96 mm to (119.2, 54.9)
- moved SW3 1.96 mm to (90.6, 73.9)
- moved SW4 1.96 mm to (109.7, 73.9)
- moved SW5 1.96 mm to (128.7, 73.9)
Connections:
- OL1 pad 1: GND -> Net-(OL1-SDA)
- OL1 pad 2: +5V -> Net-(OL1-SCL)
- OL1 pad 3: Net-(OL1-SCL) -> +5V
- OL1 pad 4: Net-(OL1-SDA) -> GND
- SW5 pad 1: Net-(U1-GPIO7/SCL) -> Net-(U1-GPIO0/TX)
- SW7 pad A: Net-(U1-GPIO26/ADC0/A0) -> Net-(U1-GPIO29/ADC3/A3)
- SW7 pad B: Net-(U1-GPIO27/ADC1/A1) -> Net-(U1-GPIO28/ADC2/A2)
- SW7 pad S1: Net-(U1-GPIO28/ADC2/A2) -> unconnected-(SW7-PadS1)
- SW7 pad S2: GND -> unconnected-(SW7-PadS2)
- U1 pad 4: Net-(OL1-SDA) -> Net-(U1-GPIO29/ADC3/A3)
- U1 pad 5: Net-(OL1-SCL) -> Net-(OL1-SDA)
- U1 pad 6: Net-(U1-GPIO7/SCL) -> Net-(OL1-SCL)
- U1 pad 7: Net-(D1-DIN) -> Net-(U1-GPIO0/TX)
Routing:
- net +5V: track 153.0 -> 15.2 mm
- net Net-(U1-GPIO0/TX): track 0.00 -> 105.9 mm
- net Net-(U1-GPIO7/SCL): track 96.0 -> 0.00 mm
- net GND: track 265.7 -> 182.9 mm
- net Net-(D1-DOUT): track 67.5 -> 0.00 mm
- net Net-(D2-DOUT): track 54.5 -> 0.00 mm
- net Net-(U1-GPIO29/ADC3/A3): track 0.00 -> 46.1 mm
- net Net-(D1-DIN): track 40.5 -> 0.00 mm
- net Net-(U1-GPIO2/SCK): track 55.5 -> 45.0 mm
- net Net-(OL1-SCL): track 23.7 -> 31.5 mm
- net Net-(U1-GPIO4/MISO): track 26.9 -> 20.4 mm
- net Net-(U1-GPIO1/RX): track 41.5 -> 35.4 mm
- net Net-(U1-GPIO28/ADC2/A2): track 48.4 -> 42.8 mm
- net Net-(U1-GPIO3/MOSI): track 29.0 -> 27.0 mm
- net Net-(OL1-SDA): track 26.0 -> 27.9 mm
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- added copper zone on B.Cu, net GND
- added copper zone on F.Cu, net GND
Other:
- board text added: "Rotary Encoder - L"
- board text added: "Rotary Encoder - R"
- board text added: "SpinKeys MK1 Made by Greg - TheTinkerersHaven Thanks to Hack Club and AMD"
- board text added: "^^^ USB-C"
- board text added: "clack clack clack"
- board text added: "click click click"
- board text added: "furries 4evr >:3"
- board text added: "guess what"
- board text added: "spinny device"
- board text added: "still a switch"
- board text added: "this one too"
- board text added: "very smart little thing right here"
- board text added: "wrong side up, buddy :)"
- board text added: "you found them all! now it's broken!"
- board text added: "yup, it's a switch."

Commit message: Small changes in naming
Parts:
- renumbered SW6 to RC1, SW7 to RC2
Routing:
- net Net-(U1-GPIO29/ADC3/A3): track 46.1 -> 44.9 mm
Changed lines of the file:
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@@
 	(net 0 "")
 	(net 1 "Net-(U1-GPIO0{slash}TX)")
-	(net 2 "unconnected-(SW6-PadS2)")
+	(net 2 "unconnected-(RC1-PadS2)")
 	(net 3 "GND")
 	(net 4 "+5V")
-	(net 5 "unconnected-(SW6-PadMP)")
-	(net 6 "unconnected-(SW6-PadS1)")
+	(net 5 "unconnected-(RC1-PadMP)")
+	(net 6 "unconnected-(RC1-PadS1)")
 	(net 7 "Net-(OL1-SDA)")
 	(net 8 "Net-(OL1-SCL)")
@@
 	(net 14 "Net-(U1-GPIO26{slash}ADC0{slash}A0)")
 	(net 15 "Net-(U1-GPIO27{slash}ADC1{slash}A1)")
-	(net 16 "unconnected-(SW7-PadMP)")
+	(net 16 "unconnected-(RC2-PadMP)")
 	(net 17 "Net-(U1-GPIO28{slash}ADC2{slash}A2)")
 	(net 18 "unconnected-(U1-3V3-Pad12)")
-	(net 19 "unconnected-(SW7-PadS2)")
-	(net 20 "unconnected-(SW7-PadS1)")
+	(net 19 "unconnected-(RC2-PadS2)")
+	(net 20 "unconnected-(RC2-PadS1)")
 	(footprint "Logo:LogoT2H-5percent"
 		(layer "F.Cu")
@@
 		(descr "Alps rotary encoder, EC11E... with switch, vertical shaft, mounting holes with circular drills, http://www.alps.com/prod/info/E/HTML/Encoder/Incremental/EC11/EC11E15204A3.html")
 		(tags "rotary encoder")
-		(property "Reference" "SW6"
+		(property "Reference" "RC1"
 			(at 2.8 -4.7 0)
 			(layer "F.SilkS")
@@
 			(layers "*.Cu" "*.Mask")
 			(remove_unused_layers no)
-			(net 5 "unconnected-(SW6-PadMP)")
+			(net 5 "unconnected-(RC1-PadMP)")
 			(pinfunction "MP")
 			(pintype "passive")
@@
 			(layers "*.Cu" "*.Mask")
 			(remove_unused_layers no)
-			(net 5 "unconnected-(SW6-PadMP)")
+			(net 5 "unconnected-(RC1-PadMP)")
 			(pinfunction "MP")
 			(pintype "passive")
@@
 			(layers "*.Cu" "*.Mask")
 			(remove_unused_layers no)
-			(net 6 "unconnected-(SW6-PadS1)")
+			(net 6 "unconnected-(RC1-PadS1)")
 			(pinfunction "S1")
 			(pintype "passive")
@@
 			(layers "*.Cu" "*.Mask")
 			(remove_unused_layers no)
-			(net 2 "unconnected-(SW6-PadS2)")
+			(net 2 "unconnected-(RC1-PadS2)")
 			(pinfunction "S2")
 			(pintype "passive")
@@
 		(descr "Alps rotary encoder, EC11E... with switch, vertical shaft, mounting holes with circular drills, http://www.alps.com/prod/info/E/HTML/Encoder/Incremental/EC11/EC11E15204A3.html")
 		(tags "rotary encoder")
-		(property "Reference" "SW7"
+		(property "Reference" "RC2"
 			(at 2.8 -4.7 0)
 			(layer "F.SilkS")
@@
 			(layers "*.Cu" "*.Mask")
 			(remove_unused_layers no)
-			(net 16 "unconnected-(SW7-PadMP)")
+			(net 16 "unconnected-(RC2-PadMP)")
 			(pinfunction "MP")
 			(pintype "passive")
@@
 			(layers "*.Cu" "*.Mask")
 			(remove_unused_layers no)
-			(net 16 "unconnected-(SW7-PadMP)")
+			(net 16 "unconnected-(RC2-PadMP)")
 			(pinfunction "MP")
 			(pintype "passive")
@@
 			(layers "*.Cu" "*.Mask")
 			(remove_unused_layers no)
-			(net 20 "unconnected-(SW7-PadS1)")
+			(net 20 "unconnected-(RC2-PadS1)")
 			(pinfunction "S1")
 			(pintype "passive")
@@
 			(layers "*.Cu" "*.Mask")
 			(remove_unused_layers no)
-			(net 19 "unconnected-(SW7-PadS2)")
+			(net 19 "unconnected-(RC2-PadS2)")
 			(pinfunction "S2")
 			(pintype "passive")
@@
 	)
 	(segment
-		(start 115.455 26.19375)
-		(end 115.455 26.045)
-		(width 0.2)
-		(layer "F.Cu")
-		(net 4)
-	)
-	(segment
 		(start 115.455 26.045)
 		(end 117.5 24)
@@
 	)
 	(segment
-		(start 99.38 33.81375)
-		(end 98.199274 33.81375)
-		(width 0.2)
-		(layer "F.Cu")
-		(net 13)
-	)
-	(segment
