File: SpinKeys-Electronics/SpinKeys.kicad_sch (KiCad schematic)
At the start: 9 parts, among them SW1 SW_Push, SW2 SW_Push, SW3 SW_Push, SW4 SW_Push, SW5 SW_Push, U1 XIAO-RP2040-DIP

Commit message: Fixed a schematic-pcb link, added fab files
Parts:
- OL1: footprint Connector_PinHeader_2.54mm:PinHeader_1x04_P2.54mm_Vertical -> OLED:SSD1306-0.91-OLED-4pin-128x32
Changed lines of the file:
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@@
 			)
 		)
-		(property "Footprint" "Connector_PinHeader_2.54mm:PinHeader_1x04_P2.54mm_Vertical"
+		(property "Footprint" "OLED:SSD1306-0.91-OLED-4pin-128x32"
 			(at 130.81 24.13 0)
 			(effects
